Commit message: v0.2.0

File: singaboat_vrx/config/component_config.xacro (robot description, xacro)
@@ -2,16 +2,16 @@
 <robot xmlns:xacro="http://ros.org/wiki/xacro" name="wam-v-components">
   <xacro:macro name="yaml_components">
+    <!-- === lidar === -->
+      <xacro:lidar name="lidar" type="16_beam" x="0.7" y="0.0" z="1.6" R="0.0" P="0.1" Y="0.0" />
     <!-- === wamv_camera === -->
-      <xacro:wamv_camera name="center_camera" x="0.875" y="0.0" P="${radians(15)}" Y="${radians(0)}" />
-      <xacro:wamv_camera name="left_camera" x="0.8" y="0.2" P="${radians(15)}" Y="${radians(0)}" />
-      <xacro:wamv_camera name="right_camera" x="0.8" y="-0.2" P="${radians(15)}" Y="${radians(0)}" />
+      <xacro:wamv_camera name="camera" visualize="False" x="0.75" y="0.0" z="1.5" R="0.0" P="${radians(15)}" Y="0.0" />
     <!-- === wamv_gps === -->
-      <xacro:wamv_gps name="gps" x="-0.85" y="0.0" />
+      <xacro:wamv_gps name="gps" x="-0.85" y="0.0" z="1.3" R="0.0" P="0.0" Y="0.0" />
     <!-- === wamv_imu === -->
-      <xacro:wamv_imu name="imu" x="-0.8" y="0.0" />
-    <!-- === lidar === -->
-      <xacro:lidar name="lidar" type="16_beam" z="1.85" P="${radians(15)}" />
+      <xacro:wamv_imu name="imu" x="-0.8" y="0.0" z="1.3" R="0.0" P="0.0" Y="0.0" />
     <!-- === wamv_ball_shooter === -->
-      <xacro:wamv_ball_shooter name="ball_shooter" x="0.55" y="-0.445" z="1.3" pitch="${radians(-45)}" yaw="${radians(0)}" />
+      <xacro:wamv_ball_shooter name="ball_shooter" x="0.55" y="-0.1" z="1.3" pitch="${radians(-45)}" yaw="0.0" />
+    <!-- === wamv_pinger === -->
+      <xacro:wamv_pinger name="pinger" position="1.0 0 -1.0" />
   </xacro:macro>
 </robot>

File: singaboat_vrx/config/thruster_config.xacro (robot description, xacro)
@@ -3,8 +3,7 @@
   <xacro:include filename="$(find wamv_description)/urdf/thrusters/engine.xacro" />
     <!-- === engine === -->
-      <xacro:engine prefix="front_left_thruster" position="1.75 0.55 0.3" orientation="0.0 0.0 -2.3562" />
-      <xacro:engine prefix="front_right_thruster" position="1.75 -0.55 0.3" orientation="0.0 0.0 2.3562" />
-      <xacro:engine prefix="rear_left_thruster" position="-1.75 0.55 0.3" orientation="0.0 0.0 -0.7854" />
-      <xacro:engine prefix="rear_right_thruster" position="-1.75 -0.55 0.3" orientation="0.0 0.0 0.7854" />
+      <xacro:engine prefix="center_thruster" position="0.0 0.0 0.318237" orientation="0.0 0.0 1.570796" />
+      <xacro:engine prefix="left_thruster" position="-2.373776 1.027135 0.318237" orientation="0.0 0.0 0.0" />
+      <xacro:engine prefix="right_thruster" position="-2.373776 -1.027135 0.318237" orientation="0.0 0.0 0.0" />
   <gazebo>
     <plugin name="wamv_gazebo_thrust" filename="libusv_gazebo_thrust_plugin.so">
@@ -12,8 +11,7 @@
       <robotNamespace>${namespace}</robotNamespace>
       <xacro:include filename="$(find wamv_gazebo)/urdf/thruster_layouts/wamv_gazebo_thruster_config.xacro" />
-        <xacro:wamv_gazebo_thruster_config name="front_left_thruster" />
-        <xacro:wamv_gazebo_thruster_config name="front_right_thruster" />
-        <xacro:wamv_gazebo_thruster_config name="rear_left_thruster" />
-        <xacro:wamv_gazebo_thruster_config name="rear_right_thruster" />
+        <xacro:wamv_gazebo_thruster_config name="center_thruster" />
+        <xacro:wamv_gazebo_thruster_config name="left_thruster" />
+        <xacro:wamv_gazebo_thruster_config name="right_thruster" />
     </plugin>
   </gazebo>

File: singaboat_vrx/urdf/singaboat.urdf (robot description, URDF)
Before this commit: robot WAM-V, 32 links, 31 joints
Links:
- removed link wamv/center_camera_link
- removed link wamv/center_camera_link_optical
- removed link wamv/center_camera_post_arm_link
- removed link wamv/center_camera_post_link
- removed link wamv/front_left_thruster_engine_link
- removed link wamv/front_left_thruster_propeller_link
- removed link wamv/front_right_thruster_engine_link
- removed link wamv/front_right_thruster_propeller_link
- removed link wamv/left_camera_link
- removed link wamv/left_camera_link_optical
- removed link wamv/left_camera_post_arm_link
- removed link wamv/left_camera_post_link
- removed link wamv/rear_left_thruster_engine_link
- removed link wamv/rear_left_thruster_propeller_link
- removed link wamv/rear_right_thruster_engine_link
- removed link wamv/rear_right_thruster_propeller_link
- removed link wamv/right_camera_link
- removed link wamv/right_camera_link_optical
- removed link wamv/right_camera_post_arm_link
- removed link wamv/right_camera_post_link
- added link wamv/camera_link, mass 0.3; collision box size=0.036 0.03 0.03; collision cylinder length=0.042 radius=0.015
- added link wamv/camera_link_optical
- added link wamv/camera_post_arm_link, mass 0.1; collision cylinder length=0.065 radius=0.008; visual mesh filename=package://vrx_gazebo/models/sensor_post/mesh/sensor_post_ar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
- added link wamv/camera_post_link, mass 0.15885000000000002; collision cylinder length=0.17650000000000002 radius=0.0076; visual cylinder length=0.17650000000000002 radius=0.0076
- added link wamv/center_thruster_engine_link, mass 15; collision box size=0.12 0.15 0.12; collision box size=0.2 0.15 0.83
- added link wamv/center_thruster_propeller_link, mass 0.5; collision cylinder length=0.18 radius=0.24; visual mesh filename=package://wamv_description/models/propeller/mesh/propeller.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
- added link wamv/left_thruster_engine_link, mass 15; collision box size=0.12 0.15 0.12; collision box size=0.2 0.15 0.83
- added link wamv/left_thruster_propeller_link, mass 0.5; collision cylinder length=0.18 radius=0.24; visual mesh filename=package://wamv_description/models/propeller/mesh/propeller.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
- added link wamv/pinger; collision box size=0.1 0.1 0.1; visual box size=0.1 0.1 0.1
- added link wamv/right_thruster_engine_link, mass 15; collision box size=0.12 0.15 0.12; collision box size=0.2 0.15 0.83
- added link wamv/right_thruster_propeller_link, mass 0.5; collision cylinder length=0.18 radius=0.24; visual mesh filename=package://wamv_description/models/propeller/mesh/propeller.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
- link wamv/lidar_post_link: mass 0.45315000000000005 -> 0.2281500000000001; geometry collision cylinder length=0.2535000000000001 radius=0.0076; visual cylinder length=0.2535000000000001 radius=0.0076
Joints:
- removed joint wamv/base_to_center_camera_post_joint
- removed joint wamv/base_to_left_camera_post_joint
- removed joint wamv/base_to_right_camera_post_joint
- removed joint wamv/center_camera_post_arm_to_center_camera_joint
- removed joint wamv/center_camera_post_to_center_camera_post_arm_joint
- removed joint wamv/center_camera_to_center_camera_link_optical_joint
- removed joint wamv/front_left_thruster_chasis_engine_joint
- removed joint wamv/front_left_thruster_engine_propeller_joint
- removed joint wamv/front_right_thruster_chasis_engine_joint
- removed joint wamv/front_right_thruster_engine_propeller_joint
- removed joint wamv/left_camera_post_arm_to_left_camera_joint
- removed joint wamv/left_camera_post_to_left_camera_post_arm_joint
- removed joint wamv/left_camera_to_left_camera_link_optical_joint
- removed joint wamv/rear_left_thruster_chasis_engine_joint
- removed joint wamv/rear_left_thruster_engine_propeller_joint
- removed joint wamv/rear_right_thruster_chasis_engine_joint
- removed joint wamv/rear_right_thruster_engine_propeller_joint
- removed joint wamv/right_camera_post_arm_to_right_camera_joint
- removed joint wamv/right_camera_post_to_right_camera_post_arm_joint
- removed joint wamv/right_camera_to_right_camera_link_optical_joint
- added joint wamv/base_to_camera_post_joint: type fixed, parent wamv/base_link, child wamv/camera_post_link, origin xyz=0.7 0.0 1.38475 rpy=0 0 0
- added joint wamv/camera_post_arm_to_camera_joint: type fixed, parent wamv/camera_post_arm_link, child wamv/camera_link, origin xyz=0.02 0 0.027 rpy=0.0 0.2617993877991494 0.0
- added joint wamv/camera_post_to_camera_post_arm_joint: type fixed, parent wamv/camera_post_link, child wamv/camera_post_arm_link, origin xyz=0.03 0 0.08825000000000008 rpy=0 0 0
- added joint wamv/camera_to_camera_link_optical_joint: type fixed, parent wamv/camera_link, child wamv/camera_link_optical, origin xyz=0 0 0 rpy=-1.5707963267948966 0 -1.5707963267948966
- added joint wamv/center_thruster_chasis_engine_joint: type revolute, parent wamv/base_link, child wamv/center_thruster_engine_link, origin xyz=0.0 0.0 0.318237 rpy=0.0 0.0 1.570796, axis 0 0 1, limit lower=-3.141592653589793 upper=3.141592653589793 effort=10 velocity=10
- added joint wamv/center_thruster_engine_propeller_joint: type continuous, parent wamv/center_thruster_engine_link, child wamv/center_thruster_propeller_link, origin xyz=-0.278156 0 -0.509371 rpy=0 0 0, axis 1 0 0, limit effort=100 velocity=100
- added joint wamv/left_thruster_chasis_engine_joint: type revolute, parent wamv/base_link, child wamv/left_thruster_engine_link, origin xyz=-2.373776 1.027135 0.318237 rpy=0.0 0.0 0.0, axis 0 0 1, limit lower=-3.141592653589793 upper=3.141592653589793 effort=10 velocity=10
- added joint wamv/left_thruster_engine_propeller_joint: type continuous, parent wamv/left_thruster_engine_link, child wamv/left_thruster_propeller_link, origin xyz=-0.278156 0 -0.509371 rpy=0 0 0, axis 1 0 0, limit effort=100 velocity=100
- added joint wamv/pinger_pinger_joint: type fixed, parent wamv/base_link, child wamv/pinger, origin xyz=1.0 0 -1.0 rpy=0 0 0
- added joint wamv/right_thruster_chasis_engine_joint: type revolute, parent wamv/base_link, child wamv/right_thruster_engine_link, origin xyz=-2.373776 -1.027135 0.318237 rpy=0.0 0.0 0.0, axis 0 0 1, limit lower=-3.141592653589793 upper=3.141592653589793 effort=10 velocity=10
- added joint wamv/right_thruster_engine_propeller_joint: type continuous, parent wamv/right_thruster_engine_link, child wamv/right_thruster_propeller_link, origin xyz=-0.278156 0 -0.509371 rpy=0 0 0, axis 1 0 0, limit effort=100 velocity=100
- joint wamv/ball_shooter_base_joint: origin xyz=0.55 -0.445 1.3 rpy=0 0 0.0 -> xyz=0.55 -0.1 1.3 rpy=0 0 0.0
- joint wamv/base_to_lidar_post_joint: origin xyz=0.6299999999999999 0.0 1.54825 rpy=0 0 0 -> xyz=0.6299999999999999 0.0 1.4232500000000001 rpy=0 0 0
- joint wamv/gps_joint: origin xyz=-0.85 0.0 1.3 rpy=0 0 0 -> xyz=-0.85 0.0 1.3 rpy=0.0 0.0 0.0
- joint wamv/imu_joint: origin xyz=-0.8 0.0 1.3 rpy=0 0 0 -> xyz=-0.8 0.0 1.3 rpy=0.0 0.0 0.0
- joint wamv/lidar_post_arm_to_lidar_joint: origin xyz=0.04 0 0.05 rpy=0 0.2617993877991494 0 -> xyz=0.04 0 0.05 rpy=0.0 0.1 0.0
- joint wamv/lidar_post_to_lidar_post_arm_joint: origin xyz=0.03 0 0.2517500000000002 rpy=0 0 0 -> xyz=0.03 0 0.12674999999999997 rpy=0 0 0
