Commit message: v0.3.0

File: singaboat_vrx/urdf/singaboat.urdf (robot description, URDF)
Before this commit: robot WAM-V, 23 links, 22 joints
Joints:
- joint wamv/ball_shooter_base_joint: origin xyz=0.55 -0.1 1.3 rpy=0 0 0.0 -> xyz=0.55 0.1 1.3 rpy=0 0 0.0

File: vrx/vrx_gazebo/worlds/stationkeeping_task.world.xacro (robot description, xacro)
@@ -24,5 +24,5 @@
       </wind_objs>
     </xacro:usv_wind_gazebo>
-  <plugin name="stationkeeping_scoring_plugin"
+    <plugin name="stationkeeping_scoring_plugin"
           filename="libstationkeeping_scoring_plugin.so">
       <vehicle>wamv</vehicle>

File: vrx/vrx_gazebo/worlds/sydneyregatta.xacro (robot description, xacro)
@@ -4,4 +4,5 @@
   <xacro:macro name="sydneyregatta">
     <scene>
+      <shadows>0</shadows>
       <sky>
         <clouds>

Commit message: Revert to v0.2.0

File: singaboat_vrx/urdf/singaboat.urdf (robot description, URDF)
Before this commit: robot WAM-V, 23 links, 22 joints
Joints:
- joint wamv/ball_shooter_base_joint: origin xyz=0.55 0.1 1.3 rpy=0 0 0.0 -> xyz=0.55 -0.1 1.3 rpy=0 0 0.0

File: vrx/vrx_gazebo/worlds/stationkeeping_task.world.xacro (robot description, xacro)
@@ -24,5 +24,5 @@
       </wind_objs>
     </xacro:usv_wind_gazebo>
-    <plugin name="stationkeeping_scoring_plugin"
+  <plugin name="stationkeeping_scoring_plugin"
           filename="libstationkeeping_scoring_plugin.so">
       <vehicle>wamv</vehicle>

File: vrx/vrx_gazebo/worlds/sydneyregatta.xacro (robot description, xacro)
@@ -4,5 +4,4 @@
   <xacro:macro name="sydneyregatta">
     <scene>
-      <shadows>0</shadows>
       <sky>
         <clouds>
